Commit message: add walking train ver1

File: robot_baseline/robot/resources/robotis_op3.urdf (robot description, URDF)
Before this commit: robot robotis_op3, 23 links, 22 joints
Links:
- link body_link: mass 0 -> 0.95181
- link head_pan_link: mass 0.01176 -> 0.001176
- link head_tilt_link: mass 0.13631 -> 0.0013631

File: robot_baseline/robot/resources/simpleplane.urdf (robot description, URDF)
Before this commit: robot simpleplane, 1 links, 0 joints
Links:
- link base_link: geometry collision box size=10.0 10.0 0.01; visual box size=10.0 10.0 0.01
